File: Schematic.kicad_sch (KiCad schematic)
At the start: 74 parts, among them J1 Screw_Terminal_01x04, J20 T44007, J21 T44007, Q1 HY1707, Q20 BC817, Q21 SUD50P06-15, U1 UC3845, U20 TCMT1108, U21 TL431M

Commit message: Layout in progress, added some rules and net classes
Parts:
- added R30: 470, Resistor_SMD:R_1206_3216Metric_Pad1.30x1.75mm_HandSolder, symbol Device:R
- added TP20, TP21, TP22, TP23, TP24, TP25, TP26, TP27, TP28, TP29, TP31, TP32, TP33, TP34: TestPoint_Alt, TestPoint:TestPoint_Loop_D3.50mm_Drill0.9mm_Beaded, symbol Connector:TestPoint_Alt
- added unit 2 of TR1
Connections:
- net Comp: now also TP25.1
- net GND: now also TP29.1, TP32.1, TP33.1
- net Isns: now also TP22.1
- net OpEm: now also TP26.1
- net SW: now also TP20.1
- net Src: now also TP21.1
- net U5_sec: now also R30.1, TP34.1
- net Vfb: now also TP24.1
- net Vin_p: now also TP31.1
- net Sec_comp_mid: now reaches C20.2, C21.1, R20.2
- net Sec_div_h: now reaches R10.1, R11.2
- net Sec_div_l: now reaches R4.2, VR1.3
- net GND_HV renamed Sec_GND
- net Sec_GND: now also R30.2, TP28.1
- net OpA renamed Sec_OpA
- net OpK renamed Sec_OpK
- net PWM_out renamed PWM
- net PWM: now also TP23.1
- net Ref_sns renamed Sec_ref_sns
- net SS_cap renamed Sec_ss_cap
- net TR_out renamed U500_tr_sec
- net Vout renamed U500_sec
- net U500_sec: now also TP27.1
- new net Pri_NR3: TR1.3
- new net Pri_NR4: TR1.4
- new net Pri_NR6: TR1.6
- new net Sec_NR10: TR1.10
- new net Sec_NR11: TR1.11
- new net Sec_NR12: TR1.12
- new net Sec_NR8: TR1.8
- new net Sec_NR9: TR1.9
- no-connect marks 2 -> 10
Other:
- moved on the sheet: C20, C21, C23, C8, D21, D22, D4, F1, J1, Q21, R10, R11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
