File: Isolated_12to450V.kicad_pcb (KiCad board)
At the start: 4 copper layers, 85 x 47.5 mm, 76 parts, among them J1 Screw_Terminal_01x04, J20 T44007, J21 T44007, Q1 HY1707, Q20 BC817, Q21 SUD50P06-15, U1 UC3845, U20 TCMT1108, U21 TL431M

Commit message: fixing templates
Other:
- board text added: "Scale 1:1"
- board text removed: "Scale 1:2"
