File: Revision History.kicad_sch (KiCad schematic)
At the start: 0 parts

Commit message: First working prototype - still not isolated
Changed lines of the file:
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@@
 		(exclude_from_sim no)
 		(at 20.32 35.56 0)
-		(size 63.5 34.29)
+		(size 63.5 154.94)
 		(margins 1.4287 1.4287 1.4287 1.4287)
 		(stroke
@@
 	(text_box "${RELEASE_BODY_1.0.1}"
 		(exclude_from_sim no)
-		(at 20.32 80.01 0)
-		(size 63.5 105.41)
+		(at 86.36 35.56 0)
+		(size 63.5 46.99)
 		(margins 1.4287 1.4287 1.4287 1.4287)
 		(stroke
@@
 	(text_box "${RELEASE_TITLE_1.0.1}"
 		(exclude_from_sim no)
-		(at 20.32 76.2 0)
+		(at 86.36 30.48 0)
 		(size 63.5 3.81)
 		(margins 1.4287 1.4287 1.4287 1.4287)

Commit message: Libraries added, revision notes and readme updated
Changed lines of the file:
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@@
 	(text_box "${RELEASE_BODY_1.0.0}"
 		(exclude_from_sim no)
-		(at 20.32 35.56 0)
+		(at 86.36 33.02 0)
 		(size 63.5 154.94)
 		(margins 1.4287 1.4287 1.4287 1.4287)
@@
 	(text_box "${RELEASE_BODY_1.0.1}"
 		(exclude_from_sim no)
-		(at 86.36 35.56 0)
-		(size 63.5 46.99)
+		(at 20.32 33.02 0)
+		(size 63.5 162.56)
 		(margins 1.4287 1.4287 1.4287 1.4287)
 		(stroke
@@
 	(text_box "${RELEASE_TITLE_1.0.0}"
 		(exclude_from_sim no)
-		(at 20.32 31.75 0)
+		(at 86.36 30.48 0)
 		(size 63.5 3.81)
 		(margins 1.4287 1.4287 1.4287 1.4287)
@@
 	(text_box "${RELEASE_TITLE_1.0.1}"
 		(exclude_from_sim no)
-		(at 86.36 30.48 0)
+		(at 20.32 30.48 0)
 		(size 63.5 3.81)
 		(margins 1.4287 1.4287 1.4287 1.4287)
