File: Revision History.kicad_sch (KiCad schematic)
At the start: 0 parts

Commit message: Preparing release
Changed lines of the file:
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@@
 		)
 	)
-	(text_box "${RELEASE_BODY_1.0.1}"
+	(text_box "${RELEASE_BODY_2.0.0}"
 		(exclude_from_sim no)
 		(at 20.32 33.02 0)
@@
 		)
 	)
-	(text_box "${RELEASE_TITLE_1.0.1}"
+	(text_box "${RELEASE_TITLE_2.0.0}"
 		(exclude_from_sim no)
 		(at 20.32 30.48 0)
