File: Revision History.kicad_sch (KiCad schematic)
At the start: 0 parts

Commit message: Updated changelog
Changed lines of the file:
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@@
 		(comment 9 "FR")
 	)
-	(text_box "${RELEASE_BODY_1.1.0}"
+	(text_box "${RELEASE_BODY_3.0.1}"
 		(exclude_from_sim no)
-		(at 29.21 35.56 0)
+		(at 20.32 35.56 0)
 		(size 63.5 111.76)
 		(margins 1.4287 1.4287 1.4287 1.4287)
@@
 		(exclude_from_sim no)
 		(at 86.36 33.02 0)
-		(size 63.5 157.48)
+		(size 63.5 118.11)
 		(margins 1.4287 1.4287 1.4287 1.4287)
 		(stroke
@@
 		)
 	)
-	(text_box "${RELEASE_TITLE_1.1.0}"
+	(text_box "${RELEASE_TITLE_3.0.1}"
 		(exclude_from_sim no)
-		(at 29.21 31.75 0)
+		(at 20.32 31.75 0)
 		(size 63.5 3.81)
 		(margins 1.4287 1.4287 1.4287 1.4287)
