File: Isolated_12to450V.kicad_sch (KiCad schematic)
At the start: 0 parts

Commit message: Preparing release
Other:
- note added: "Status: ${VARIANT}"
- note removed: "${SHEET_NAME_10}"
- note removed: "${SHEET_NAME_5}"
- note removed: "${SHEET_NAME_6}"
- note removed: "${SHEET_NAME_7}"
- note removed: "${SHEET_NAME_8}"
- note removed: "${SHEET_NAME_9}"
- note removed: "10"
- note removed: "5"
- note removed: "6"
- note removed: "7"
- note removed: "8"
- note removed: "9"
- note removed: "Variant: ${VARIANT}"

Commit message: layout update started
Changed lines of the file:
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@@
-		)
-	)
-	(text_box "DRAFT - Early concept stage, schematic drafted.\n\nPRELIMINARY - Minor schematic changes are expected, ready for layout planning.\n\nCHECKED - DRC completed, schematic and layout ready for review.\n\nRELEASED - Design ready for manufacturing."
-		(exclude_from_sim no)
-		(at 25.4 196.85 0)
-		(size 165.1 44.45)
-		(margins 2 2 2 2)
-		(stroke
-			(width 0.508)
-			(type solid)
-			(color 132 132 132 1)
-		)
-		(fill
-			(type color)
-			(color 200 200 200 1)
-		)
-		(effects
-			(font
-				(face "Arial")
-				(size 3.048 3.048)
-				(color 0 0 0 1)
-			)
-			(justify left)
 		)
 	)
