File: PerfBoard.kicad_sch (KiCad schematic)
At the start: 252 parts

Commit message: ERC/DRC completed
Parts:
- added H101, H102, H103, H104: MountingHole, MountingHole:MountingHole_3.2mm_M3, symbol Mechanical:MountingHole
